Commit message: up

File: install/robot_description/share/robot_description/urdf/gazebo.xacro (robot description, xacro)
@@ -1,206 +1 @@
-<?xml version="1.0"?>
-<!--
-  gazebo.xacro - Gazebo simulation plugins and properties.
-  This file adds Gazebo-specific elements to the robot model:
-    1. Friction coefficients for wheels and caster
-    2. Differential drive controller plugin (simulates ESP32 + motors)
-    3. Lidar sensor plugin (simulates RPLidar C1)
-    4. IMU sensor plugin
-    5. Camera sensor plugin
-  When running in Gazebo, these plugins replace the real hardware:
-    - diff_drive plugin publishes /odom and subscribes to /cmd_vel
-    - lidar plugin publishes /scan
-    - imu plugin publishes /imu/data
-  Usage:
-    Included by robot.urdf.xacro. Only active when loading in Gazebo.
-    Does NOT affect real robot operation.
--->
-<robot xmlns:xacro="http://www.ros.org/wiki/xacro">
-  <!-- ============= Gazebo Material Colors ================= -->
-  <gazebo reference="base_link">
-    <material>Gazebo/Blue</material>
-  </gazebo>
-  <gazebo reference="left_wheel">
-    <material>Gazebo/DarkGrey</material>
-    <mu1>1.0</mu1>
-    <mu2>1.0</mu2>
-    <kp>1000000.0</kp>
-    <kd>100.0</kd>
-  </gazebo>
-  <gazebo reference="right_wheel">
-    <material>Gazebo/DarkGrey</material>
-    <mu1>1.0</mu1>
-    <mu2>1.0</mu2>
-    <kp>1000000.0</kp>
-    <kd>100.0</kd>
-  </gazebo>
-  <gazebo reference="rear_caster_wheel">
-    <material>Gazebo/Grey</material>
-    <mu1>0.001</mu1>
-    <mu2>0.001</mu2>
-    <kp>1000000.0</kp>
-    <kd>100.0</kd>
-  </gazebo>
-  <!-- ============= Differential Drive Plugin ============== -->
-  <!--
-    Simulates the ESP32 + BTS7960 motor controller.
-    In Gazebo, this plugin:
-      - Subscribes to /cmd_vel (geometry_msgs/Twist)
-      - Publishes /odom (nav_msgs/Odometry)
-      - Publishes TF: odom -> base_footprint
-    Parameters match the real robot's kinematics:
-      wheel_separation: distance between left and right wheels
-      wheel_diameter: diameter of drive wheels
-  -->
-  <gazebo>
-    <plugin name="diff_drive" filename="libgazebo_ros_diff_drive.so">
-      <ros>
-        <namespace>/</namespace>
-      </ros>
-      <!-- Wheels -->
-      <left_joint>left_wheel_joint</left_joint>
-      <right_joint>right_wheel_joint</right_joint>
-      <!-- Kinematics -->
-      <wheel_separation>0.30</wheel_separation>
-      <wheel_diameter>0.066</wheel_diameter>
-      <!-- Limits -->
-      <max_wheel_torque>20.0</max_wheel_torque>
-      <max_wheel_acceleration>1.0</max_wheel_acceleration>
-      <!-- Output -->
-      <publish_odom>true</publish_odom>
-      <publish_odom_tf>true</publish_odom_tf>
-      <publish_wheel_tf>true</publish_wheel_tf>
-      <odometry_frame>odom</odometry_frame>
-      <robot_base_frame>base_footprint</robot_base_frame>
-      <update_rate>30</update_rate>
-    </plugin>
-  </gazebo>
-  <!-- ============= RPLidar C1 Gazebo Plugin =============== -->
-  <!--
-    Simulates the RPLidar C1M1 in Gazebo.
-    Publishes /scan (sensor_msgs/LaserScan) matching real C1 specs:
-      - 12m max range
-      - 360 degrees
-      - ~8000 points/s at 10Hz
-  -->
-  <gazebo reference="laser">
-    <sensor type="ray" name="rplidar_c1">
-      <pose>0 0 0 0 0 0</pose>
-      <visualize>true</visualize>
-      <update_rate>10</update_rate>
-      <ray>
-        <scan>
-          <horizontal>
-            <samples>720</samples>
-            <resolution>1</resolution>
-            <min_angle>-3.14159</min_angle>
-            <max_angle>3.14159</max_angle>
-          </horizontal>
-        </scan>
-        <range>
-          <min>0.12</min>
-          <max>12.0</max>
-          <resolution>0.01</resolution>
-        </range>
-        <noise>
-          <type>gaussian</type>
-          <mean>0.0</mean>
-          <stddev>0.01</stddev>
-        </noise>
-      </ray>
-      <plugin name="lidar_controller" filename="libgazebo_ros_ray_sensor.so">
-        <ros>
-          <remapping>~/out:=scan</remapping>
-        </ros>
-        <output_type>sensor_msgs/LaserScan</output_type>
-        <frame_name>laser</frame_name>
-      </plugin>
-    </sensor>
-  </gazebo>
-  <!-- ============= IMU Gazebo Plugin ====================== -->
-  <gazebo reference="imu_link">
-    <sensor type="imu" name="imu_sensor">
-      <always_on>true</always_on>
-      <update_rate>100</update_rate>
-      <imu>
-        <angular_velocity>
-          <x>
-            <noise type="gaussian">
-              <mean>0.0</mean>
-              <stddev>0.001</stddev>
-            </noise>
-          </x>
-          <y>
-            <noise type="gaussian">
-              <mean>0.0</mean>
-              <stddev>0.001</stddev>
-            </noise>
-          </y>
-          <z>
-            <noise type="gaussian">
-              <mean>0.0</mean>
-              <stddev>0.001</stddev>
-            </noise>
-          </z>
-        </angular_velocity>
-        <linear_acceleration>
-          <x>
-            <noise type="gaussian">
-              <mean>0.0</mean>
-              <stddev>0.01</stddev>
-            </noise>
-          </x>
-          <y>
-            <noise type="gaussian">
-              <mean>0.0</mean>
-              <stddev>0.01</stddev>
-            </noise>
-          </y>
-          <z>
-            <noise type="gaussian">
-              <mean>0.0</mean>
-              <stddev>0.01</stddev>
-            </noise>
-          </z>
-        </linear_acceleration>
-      </imu>
-      <plugin name="imu_plugin" filename="libgazebo_ros_imu_sensor.so">
-        <ros>
-          <remapping>~/out:=imu/data</remapping>
-        </ros>
-        <frame_name>imu_link</frame_name>
-      </plugin>
-    </sensor>
-  </gazebo>
-  <!-- ============= Camera Gazebo Plugin =================== -->
-  <gazebo reference="camera_link">
-    <sensor type="camera" name="usb_camera">
-      <update_rate>30</update_rate>
-      <camera name="ugreen_cam">
-        <horizontal_fov>1.3962634</horizontal_fov>
-        <image>
-          <width>640</width>
-          <height>480</height>
-          <format>R8G8B8</format>
-        </image>
-        <clip>
-          <near>0.02</near>
-          <far>300</far>
-        </clip>
-        <noise>
-          <type>gaussian</type>
-          <mean>0.0</mean>
-          <stddev>0.007</stddev>
-        </noise>
-      </camera>
-      <plugin name="camera_controller" filename="libgazebo_ros_camera.so">
-        <ros>
-          <remapping>~/image_raw:=camera/image_raw</remapping>
-          <remapping>~/camera_info:=camera/camera_info</remapping>
-        </ros>
-        <camera_name>camera</camera_name>
-        <frame_name>camera_optical_frame</frame_name>
-      </plugin>
-    </sensor>
-  </gazebo>
-</robot>
+/home/robot/robot_ws/src/robot_description/urdf/gazebo.xacro

File: install/robot_description/share/robot_description/urdf/macros.xacro (robot description, xacro)
@@ -1,165 +1 @@
-<?xml version="1.0"?>
-<!--
-  macros.xacro - Reusable Xacro macros for robot components.
-  Macros defined:
-    1. drive_wheel   - A drive wheel with continuous joint (for odometry)
-    2. caster_wheel  - A passive caster wheel (fixed or ball joint)
-    3. encoder       - An encoder mounted on a wheel axis
-    4. inertial_cylinder - Helper for cylinder inertia
-  Usage:
-    Included by robot.urdf.xacro. Call with:
-      <xacro:drive_wheel prefix="left" x="0" y="0.15" .../>
--->
-<robot xmlns:xacro="http://www.ros.org/wiki/xacro">
-  <!-- ============= Inertia helpers ======================== -->
-  <!-- Cylinder inertia (aligned along Z axis) -->
-  <xacro:macro name="cylinder_inertia" params="mass radius length">
-    <inertial>
-      <mass value="${mass}"/>
-      <inertia
-        ixx="${(1.0/12.0) * mass * (3*radius*radius + length*length)}"
-        ixy="0" ixz="0"
-        iyy="${(1.0/12.0) * mass * (3*radius*radius + length*length)}"
-        iyz="0"
-        izz="${(1.0/2.0) * mass * radius * radius}"/>
-    </inertial>
-  </xacro:macro>
-  <!-- Box inertia -->
-  <xacro:macro name="box_inertia" params="mass x y z">
-    <inertial>
-      <mass value="${mass}"/>
-      <inertia
-        ixx="${(1.0/12.0) * mass * (y*y + z*z)}"
-        ixy="0" ixz="0"
-        iyy="${(1.0/12.0) * mass * (x*x + z*z)}"
-        iyz="0"
-        izz="${(1.0/12.0) * mass * (x*x + y*y)}"/>
-    </inertial>
-  </xacro:macro>
-  <!-- Sphere inertia -->
-  <xacro:macro name="sphere_inertia" params="mass radius">
-    <inertial>
-      <mass value="${mass}"/>
-      <inertia
-        ixx="${(2.0/5.0) * mass * radius * radius}"
-        ixy="0" ixz="0"
-        iyy="${(2.0/5.0) * mass * radius * radius}"
-        iyz="0"
-        izz="${(2.0/5.0) * mass * radius * radius}"/>
-    </inertial>
-  </xacro:macro>
-  <!-- ============= Drive Wheel Macro ====================== -->
-  <!--
-    Creates a drive wheel link + continuous joint.
-    The continuous joint allows rotation (needed for odometry).
-    Parameters:
-      prefix    : "left" or "right"
-      wheel_radius : wheel radius in meters
-      wheel_width  : wheel thickness in meters
-      wheel_mass   : wheel mass in kg
-      x_offset     : X position relative to base_link center
-      y_offset     : Y position relative to base_link center
-      z_offset     : Z position relative to base_link center
-  -->
-  <xacro:macro name="drive_wheel" params="prefix wheel_radius wheel_width wheel_mass x_offset y_offset z_offset">
-    <!-- Wheel link -->
-    <link name="${prefix}_wheel">
-      <visual>
-        <geometry>
-          <cylinder radius="${wheel_radius}" length="${wheel_width}"/>
-        </geometry>
-        <material name="wheel_gray"/>
-        <!-- Rotate cylinder to align with Y axis (wheel orientation) -->
-        <origin xyz="0 0 0" rpy="${pi/2} 0 0"/>
-      </visual>
-      <collision>
-        <geometry>
-          <cylinder radius="${wheel_radius}" length="${wheel_width}"/>
-        </geometry>
-        <origin xyz="0 0 0" rpy="${pi/2} 0 0"/>
-      </collision>
-      <xacro:cylinder_inertia mass="${wheel_mass}" radius="${wheel_radius}" length="${wheel_width}"/>
-    </link>
-    <!-- Continuous joint: wheel can rotate freely -->
-    <!-- When ESP32 provides odometry, this joint receives /joint_states -->
-    <joint name="${prefix}_wheel_joint" type="continuous">
-      <parent link="base_link"/>
-      <child  link="${prefix}_wheel"/>
-      <origin xyz="${x_offset} ${y_offset} ${z_offset}" rpy="0 0 0"/>
-      <axis xyz="0 1 0"/>
-      <!-- Friction for Gazebo simulation -->
-      <dynamics damping="0.1" friction="0.1"/>
-    </joint>
-  </xacro:macro>
-  <!-- ============= Caster Wheel Macro ===================== -->
-  <!--
-    Creates a passive caster wheel (sphere) at the rear.
-    Uses a fixed joint (no actuation, just for physical support).
-    Parameters:
-      prefix        : "front" or "rear"
-      caster_radius : caster ball radius in meters
-      caster_mass   : caster mass in kg
-      x_offset      : X position relative to base_link
-      y_offset      : Y position relative to base_link
-      z_offset      : Z position relative to base_link
-  -->
-  <xacro:macro name="caster_wheel" params="prefix caster_radius caster_mass x_offset y_offset z_offset">
-    <link name="${prefix}_caster_wheel">
-      <visual>
-        <geometry>
-          <sphere radius="${caster_radius}"/>
-        </geometry>
-        <material name="caster_bronze"/>
-        <origin xyz="0 0 0" rpy="0 0 0"/>
-      </visual>
-      <collision>
-        <geometry>
-          <sphere radius="${caster_radius}"/>
-        </geometry>
-        <origin xyz="0 0 0" rpy="0 0 0"/>
-      </collision>
-      <xacro:sphere_inertia mass="${caster_mass}" radius="${caster_radius}"/>
-    </link>
-    <joint name="${prefix}_caster_joint" type="fixed">
-      <parent link="base_link"/>
-      <child  link="${prefix}_caster_wheel"/>
-      <origin xyz="${x_offset} ${y_offset} ${z_offset}" rpy="0 0 0"/>
-    </joint>
-  </xacro:macro>
-  <!-- ============= Encoder Macro ========================== -->
-  <!--
-    Creates an encoder link attached to the wheel axis.
-    The encoder itself doesn't rotate; it's mounted on the chassis
-    and reads the wheel's rotation.
-    Parameters:
-      prefix    : "left" or "right"
-      enc_x, enc_y, enc_z : dimensions of encoder box
-      enc_mass  : encoder mass
-      x_offset  : position relative to base_link
-      y_offset  : position relative to base_link
-      z_offset  : position relative to base_link
-  -->
-  <xacro:macro name="encoder" params="prefix enc_x enc_y enc_z enc_mass x_offset y_offset z_offset">
-    <link name="${prefix}_encoder">
-      <visual>
-        <geometry>
-          <box size="${enc_x} ${enc_y} ${enc_z}"/>
-        </geometry>
-        <material name="encoder_yellow"/>
-        <origin xyz="0 0 0" rpy="0 0 0"/>
-      </visual>
-      <collision>
-        <geometry>
-          <box size="${enc_x} ${enc_y} ${enc_z}"/>
-        </geometry>
-        <origin xyz="0 0 0" rpy="0 0 0"/>
-      </collision>
-      <xacro:box_inertia mass="${enc_mass}" x="${enc_x}" y="${enc_y}" z="${enc_z}"/>
-    </link>
-    <joint name="${prefix}_encoder_joint" type="fixed">
-      <parent link="base_link"/>
-      <child  link="${prefix}_encoder"/>
-      <origin xyz="${x_offset} ${y_offset} ${z_offset}" rpy="0 0 0"/>
-    </joint>
-  </xacro:macro>
-</robot>
+/home/robot/robot_ws/src/robot_description/urdf/macros.xacro

File: install/robot_description/share/robot_description/urdf/materials.xacro (robot description, xacro)
@@ -1,51 +1 @@
-<?xml version="1.0"?>
-<!--
-  materials.xacro - Color definitions for the robot model.
-  Usage:
-    Included by robot.urdf.xacro via <xacro:include filename="materials.xacro"/>
-  Convention:
-    Each material has a name and an RGBA color (0-1 range).
-    These are used in <material> tags inside <visual> elements.
--->
-<robot xmlns:xacro="http://www.ros.org/wiki/xacro">
-  <!-- Chassis: dark blue -->
-  <material name="chassis_blue">
-    <color rgba="0.15 0.15 0.6 1.0"/>
-  </material>
-  <!-- Wheels: dark rubber gray -->
-  <material name="wheel_gray">
-    <color rgba="0.2 0.2 0.2 1.0"/>
-  </material>
-  <!-- Caster wheel: bronze -->
-  <material name="caster_bronze">
-    <color rgba="0.6 0.4 0.2 1.0"/>
-  </material>
-  <!-- RPLidar: dark gray cylinder -->
-  <material name="lidar_dark">
-    <color rgba="0.15 0.15 0.15 1.0"/>
-  </material>
-  <!-- Camera: matte black -->
-  <material name="camera_black">
-    <color rgba="0.05 0.05 0.05 1.0"/>
-  </material>
-  <!-- Raspberry Pi: PCB green -->
-  <material name="rpi_green">
-    <color rgba="0.0 0.5 0.2 1.0"/>
-  </material>
-  <!-- IMU: orange -->
-  <material name="imu_orange">
-    <color rgba="0.9 0.5 0.0 1.0"/>
-  </material>
-  <!-- Battery: red -->
-  <material name="battery_red">
-    <color rgba="0.7 0.1 0.1 1.0"/>
-  </material>
-  <!-- Encoder: yellow -->
-  <material name="encoder_yellow">
-    <color rgba="0.9 0.8 0.0 1.0"/>
-  </material>
-  <!-- Generic white -->
-  <material name="white">
-    <color rgba="1.0 1.0 1.0 1.0"/>
-  </material>
-</robot>
+/home/robot/robot_ws/src/robot_description/urdf/materials.xacro
